Commit message: Training works, Robot doesn't learn

File: src/holosoma/holosoma/data/robots/star/star_18dof.urdf (robot description, URDF)
Before this commit: robot star_18dof, 17 links, 16 joints
Links:
- removed link head_link
- removed link left_foot_contact_point
- removed link right_foot_contact_point
- removed link torso_link
- added link head, mass 2.0; collision sphere radius=0.09; visual sphere radius=0.09
- added link lower_waist, mass 4.0; collision capsule length=0.12 radius=0.06; visual capsule length=0.12 radius=0.06
- added link torso, mass 10.0; collision capsule length=0.14 radius=0.07; visual capsule length=0.14 radius=0.07
- added link upper_waist, mass 5.0; collision capsule length=0.12 radius=0.06; visual capsule length=0.12 radius=0.06
- link left_ankle_pitch_link: mass 0.6 -> 1.5
- link left_ankle_roll_link: mass 0.3 -> 0.5
- link left_hip_pitch_link: mass 1.5 -> 6.0; geometry collision capsule length=0.34 radius=0.06; visual capsule length=0.34 radius=0.06
- link left_hip_roll_link: mass 0.5 -> 1.0
- link left_hip_yaw_link: mass 0.5 -> 1.0
- link left_knee_link: mass 1.5 -> 4.0; geometry collision capsule length=0.3 radius=0.049; visual capsule length=0.3 radius=0.049
- link pelvis: mass 5.0 -> 24.227; geometry collision capsule length=0.14 radius=0.09; visual capsule length=0.14 radius=0.09
- link right_ankle_pitch_link: mass 0.6 -> 1.5
- link right_ankle_roll_link: mass 0.3 -> 0.5
- link right_hip_pitch_link: mass 1.5 -> 6.0; geometry collision capsule length=0.34 radius=0.06; visual capsule length=0.34 radius=0.06
- link right_hip_roll_link: mass 0.5 -> 1.0
- link right_hip_yaw_link: mass 0.5 -> 1.0
- link right_knee_link: mass 1.5 -> 4.0; geometry collision capsule length=0.3 radius=0.049; visual capsule length=0.3 radius=0.049
Joints:
- removed joint head_joint
- removed joint left_foot_contact_joint
- removed joint right_foot_contact_joint
- removed joint torso_joint
- added joint head_fixed: type fixed, parent torso, child head, origin xyz=0 0 0.19 rpy=0 0 0
- added joint lower_waist_fixed: type fixed, parent upper_waist, child lower_waist, origin xyz=0 0 -0.14 rpy=0 0 0
- added joint pelvis_fixed: type fixed, parent lower_waist, child pelvis, origin xyz=0.0 0 -0.165 rpy=0 0 0
- added joint upper_waist_fixed: type fixed, parent torso, child upper_waist, origin xyz=-0.01 0 -0.12 rpy=0 0 0
- joint left_ankle_pitch_joint: limit lower=-0.5236 upper=0.5236 effort=262 velocity=37.0 -> lower=-0.5236 upper=0.5236 effort=262.0 velocity=37.0; origin xyz=0.04 0 0 rpy=0 0 0 -> xyz=0.04 0 -0.02 rpy=0 0 0
- joint left_ankle_roll_joint: limit lower=-0.6981 upper=0.4363 effort=131 velocity=37.0 -> lower=-0.6981 upper=0.4363 effort=131.0 velocity=37.0
- joint left_hip_pitch_joint: limit lower=-0.5236 upper=0.6981 effort=298 velocity=20.0 -> lower=-0.5236 upper=0.6981 effort=298.0 velocity=20.0
- joint left_hip_roll_joint: limit lower=-0.3491 upper=0.1396 effort=351 velocity=20.0 -> lower=-0.3491 upper=0.1396 effort=351.0 velocity=20.0
- joint left_hip_yaw_joint: limit lower=-0.8727 upper=0.3491 effort=351 velocity=32.0 -> lower=-0.8727 upper=0.3491 effort=351.0 velocity=32.0; origin xyz=0 0.1 -0.205 rpy=0 0 0 -> xyz=0 0.1 -0.04 rpy=0 0 0; parent torso_link -> pelvis
- joint left_knee_joint: limit lower=-0.0873 upper=1.7453 effort=420 velocity=20.0 -> lower=-0.0873 upper=1.7453 effort=420.0 velocity=20.0
- joint right_ankle_pitch_joint: limit lower=-0.5236 upper=0.5236 effort=262 velocity=37.0 -> lower=-0.5236 upper=0.5236 effort=262.0 velocity=37.0; origin xyz=0.04 0 0 rpy=0 0 0 -> xyz=0.04 0 -0.02 rpy=0 0 0
- joint right_ankle_roll_joint: limit lower=-0.6981 upper=0.4363 effort=131 velocity=37.0 -> lower=-0.6981 upper=0.4363 effort=131.0 velocity=37.0
- joint right_hip_pitch_joint: limit lower=-0.5236 upper=0.6981 effort=298 velocity=20.0 -> lower=-0.5236 upper=0.6981 effort=298.0 velocity=20.0
- joint right_hip_roll_joint: limit lower=-0.3491 upper=0.1396 effort=351 velocity=20.0 -> lower=-0.3491 upper=0.1396 effort=351.0 velocity=20.0
- joint right_hip_yaw_joint: limit lower=-0.8727 upper=0.3491 effort=351 velocity=32.0 -> lower=-0.8727 upper=0.3491 effort=351.0 velocity=32.0; origin xyz=0 -0.1 -0.205 rpy=0 0 0 -> xyz=0 -0.1 -0.04 rpy=0 0 0; parent torso_link -> pelvis
- joint right_knee_joint: limit lower=-0.0873 upper=1.7453 effort=420 velocity=20.0 -> lower=-0.0873 upper=1.7453 effort=420.0 velocity=20.0

Commit message: Robot falls early

File: src/holosoma/holosoma/data/robots/star/star_18dof.urdf (robot description, URDF)
Before this commit: robot star_18dof, 17 links, 16 joints
Joints:
- joint left_hip_roll_joint: axis -1 0 0 -> 1 0 0
- joint left_hip_yaw_joint: axis 0 0 -1 -> 0 0 1
